File: NRG Detachable Steering Wheel Insert/NRG Detachable Steering Wheel Insert.kicad_sch (KiCad schematic)
At the start: 18 parts, among them J1 Conn_01x01, J10 Conn_01x01, J11 Conn_01x01, J12 Conn_01x01, J13 Conn_01x01, J14 Conn_01x01, J15 Conn_01x01, J16 Conn_01x01, J2 Conn_01x01, J3 Conn_01x01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

Commit message: Updating the steering wheel insert to not touch the metal of the steering wheel.
Parts:
- J1, J2, J3, J4: Manufacturer (none) -> Mill-Max Manufacturing Corp.; Part Num (none) -> 0921-0-15-20-76-14-11-0; Vendor (none) -> Digi-Key; Vendor Part Num (none) -> ED1656-ND
Changed lines of the file:
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@@
+      (effects (font (size 1.27 1.27)) hide)
+    )
+    (property "Description" "Contact Spring Through Hole" (id 4) (at 55.88 48.26 0)
+      (effects (font (size 1.27 1.27)) hide)
+    )
+    (property "Manufacturer" "Mill-Max Manufacturing Corp." (id 5) (at 55.88 48.26 0)
+      (effects (font (size 1.27 1.27)) hide)
+    )
+    (property "Part Num" "0921-0-15-20-76-14-11-0" (id 6) (at 55.88 48.26 0)
+      (effects (font (size 1.27 1.27)) hide)
+    )
+    (property "Vendor" "Digi-Key" (id 7) (at 55.88 48.26 0)
+      (effects (font (size 1.27 1.27)) hide)
+    )
+    (property "Vendor Part Num" "ED1656-ND" (id 8) (at 55.88 48.26 0)
       (effects (font (size 1.27 1.27)) hide)
     )
@@
       (effects (font (size 1.27 1.27)) hide)
     )
+    (property "Description" "Contact Spring Through Hole" (id 4) (at 55.88 57.785 0)
+      (effects (font (size 1.27 1.27)) hide)
+    )
+    (property "Manufacturer" "Mill-Max Manufacturing Corp." (id 5) (at 55.88 57.785 0)
+      (effects (font (size 1.27 1.27)) hide)
+    )
+    (property "Part Num" "0921-0-15-20-76-14-11-0" (id 6) (at 55.88 57.785 0)
+      (effects (font (size 1.27 1.27)) hide)
+    )
+    (property "Vendor" "Digi-Key" (id 7) (at 55.88 57.785 0)
+      (effects (font (size 1.27 1.27)) hide)
+    )
+    (property "Vendor Part Num" "ED1656-ND" (id 8) (at 55.88 57.785 0)
+      (effects (font (size 1.27 1.27)) hide)
+    )
     (pin "1")
   )
@@
       (effects (font (size 1.27 1.27)) hide)
     )
+    (property "Description" "Contact Spring Through Hole" (id 4) (at 55.88 66.675 0)
+      (effects (font (size 1.27 1.27)) hide)
+    )
+    (property "Manufacturer" "Mill-Max Manufacturing Corp." (id 5) (at 55.88 66.675 0)
+      (effects (font (size 1.27 1.27)) hide)
+    )
+    (property "Part Num" "0921-0-15-20-76-14-11-0" (id 6) (at 55.88 66.675 0)
+      (effects (font (size 1.27 1.27)) hide)
+    )
+    (property "Vendor" "Digi-Key" (id 7) (at 55.88 66.675 0)
+      (effects (font (size 1.27 1.27)) hide)
+    )
+    (property "Vendor Part Num" "ED1656-ND" (id 8) (at 55.88 66.675 0)
+      (effects (font (size 1.27 1.27)) hide)
+    )
     (pin "1")
   )
@@
       (effects (font (size 1.27 1.27)) hide)
     )
+    (property "Description" "Contact Spring Through Hole" (id 4) (at 55.88 38.735 0)
+      (effects (font (size 1.27 1.27)) hide)
+    )
+    (property "Manufacturer" "Mill-Max Manufacturing Corp." (id 5) (at 55.88 38.735 0)
+      (effects (font (size 1.27 1.27)) hide)
+    )
+    (property "Part Num" "0921-0-15-20-76-14-11-0" (id 6) (at 55.88 38.735 0)
+      (effects (font (size 1.27 1.27)) hide)
+    )
+    (property "Vendor" "Digi-Key" (id 7) (at 55.88 38.735 0)
+      (effects (font (size 1.27 1.27)) hide)
+    )
+    (property "Vendor Part Num" "ED1656-ND" (id 8) (at 55.88 38.735 0)
+      (effects (font (size 1.27 1.27)) hide)
+    )
