File: Corolla 2006 DBW Stock Harness to EMU Black/Corolla 2006 DBW Stock Harness to EMU Black.kicad_sch (KiCad schematic)
At the start: 13 parts

Commit message: Commit whatever changes are in the repository.
Parts:
- added D? (x3): NO STUFF, symbol Device:D
- J?: symbol Connector_Generic:Conn_01x31 -> toyota:Corolla_2006_DBW_ECU
- J?: symbol Connector_Generic:Conn_01x34 -> toyota:Corolla_2006_DBW_ECU
- J? (x2): symbol Connector_Generic:Conn_01x35 -> toyota:Corolla_2006_DBW_ECU
Connections:
- net AC CLUTCH: now also J?.C2 (A/C_Mag_Clutch_Relay); no longer J?.2 (Pin_2)
- net AC ENABLE: now also J?.C28 (A/C_Enable_SW); no longer J?.28 (Pin_28)
- net AC EVAP THERM: now also J?.C32 (A/C_Evap_Thermistor); no longer J?.32 (Pin_32)
- net ACCEL TPS 1: now also J?.D22 (Accel_Position_1_Signal); no longer J?.22 (Pin_22)
- net ACCEL TPS 2: now also J?.D23 (Accel_Position_2_Signal); no longer J?.23 (Pin_23)
- net BAT 12V: now also J?.D3 (EFI_Fuse_(Battery)), D?.1 (K), D?.1 (K); no longer J?.6 (Pin_6)
- net CAM POS: now also J?.B24 (Camshaft_Position_Sensor+); no longer J?.24 (Pin_24)
- net COOLANT TEMP: now also J?.A19 (Coolant_Temp_Sensor); no longer J?.19 (Pin_19)
- net CRANK POS: now also J?.B25 (Crankshaft_Position_Sensor+); no longer J?.25 (Pin_25)
- net DBW M+: now also J?.B4 (Drive_By_Wire_(DBW)_Motor+); no longer J?.4 (Pin_4)
- net DBW M-: now also J?.B3 (Drive_By_Wire_(DBW)_Motor-); no longer J?.3 (Pin_3)
- net ECU GND: now also J?.B35 (Chassis_Ground), D?.2 (A); no longer J?.35 (Pin_35)
- net FUEL PUMP: now also J?.D10 (Fuel_Pump_Relay); no longer J?.10 (Pin_10)
- net IGN COIL 1: now also J?.A8 (Ignition_Coil_1); no longer J?.8 (Pin_8)
- net IGN COIL 2: now also J?.A9 (Ignition_Coil_2); no longer J?.9 (Pin_9)
- net IGN COIL 3: now also J?.A10 (Ignition_Coil_3); no longer J?.10 (Pin_10)
- net IGN COIL 4: now also J?.A11 (Ignition_Coil_4); no longer J?.11 (Pin_11)
- net INJ 1: now also J?.A1 (Injector_1); no longer J?.1 (Pin_1)
- net INJ 2: now also J?.A2 (Injector_2); no longer J?.2 (Pin_2)
- net INJ 3: now also J?.A3 (Injector_3); no longer J?.3 (Pin_3)
- net INJ 4: now also J?.A4 (Injector_4); no longer J?.4 (Pin_4)
- net INTAKE TEMP: now also J?.A20 (MAF_Thermistor); no longer J?.20 (Pin_20)
- net KNOCK SENS: now also J?.B1 (Knock_Sensor+); no longer J?.1 (Pin_1)
- net PS LOW: now also J?.B8 (Power_Steering_Fluid_Low); no longer J?.8 (Pin_8)
- net PWR GND 1: no longer J?.27 (Power_Ground), J?.6 (Pin_6)
- net RAD FAN: now also J?.B16 (Radiator_Fan_On/Off); no longer J?.16 (Pin_16)
- net SENS GND 1: no longer J?.28 (Pin_28), J?.29 (Sensor_Ground)
- net SENS PWR 1: now also J?.A18 (Throttle_Sensor_Power); no longer J?.18 (Pin_18)
- net SENS PWR 2: now also J?.D26 (Accel_Position_1_V+), J?.D27 (Accel_Position_2_V+); no longer J?.26 (Pin_26), J?.27 (Pin_27)
- net STOP LAMP: now also J?.C19 (Stop_Lamp_Active); no longer J?.19 (Pin_19)
- net SW 12V: now also J?.A13 (Camsgaft_Timing_Control+_(VVT)), J?.A14 (Radiator_Fan_High/Low), J?.D1 (EFI2_Fuse_(After_EFI_Relay)), D?.2 (A); no longer J?.1 (Pin_1), J?.13 (Pin_13), J?.14 (Pin_14)
- net TB TPS 1: now also J?.A21 (Throttle_Body_Position_Sensor_1); no longer J?.21 (Pin_21)
- net TB TPS 2: now also J?.A31 (Throttle_Body_Position_Sensor_2); no longer J?.31 (Pin_31)
- net VSS: now also J?.C17 (Speed_Sensor); no longer J?.17 (Pin_17)
- net VVT SOL: now also J?.A12 (Camshaft_Timing_Control-_(VVT)); no longer J?.12 (Pin_12)
- net PWR GND 2 renamed PWR GND
- net PWR GND: now also J?.24 (Power_Ground), J?.27 (Power_Ground), J?.A6 (Power_Ground), J?.A7 (Power_Ground), J?.B17 (Drive_By_Wire_(DBW)_Shield), J?.B2 (Power_Ground), J?.B6 (Power_Ground), J?.B7 (Power_Ground), J?.C33 (A/C_Switch_Indicator), J?.D15 (Power_Ground), D?.1 (K); no longer J?.2 (Pin_2)
- removed net PWR GND 3: J?.24 (Power_Ground), J?.6 (Pin_6)
- removed net SENS GND 2: J?.28 (Pin_28), J?.33 (Pin_33), J?.38 (Sensor_Ground)
- removed net SENS GND 3: J?.28 (Pin_28), J?.29 (Pin_29), J?.39 (Sensor_Ground)
- new net: J?.D8 (EFI_Relay_Coil), J?.D9 (Ignition_Switch_Signal)
- new net: D?.2 (A), J?.C6 (ETCS_Fuse_(Battery))
- new net SENS GND: J?.29 (Sensor_Ground), J?.38 (Sensor_Ground), J?.39 (Sensor_Ground), J?.A28 (Signal_Ground), J?.B28 (Knock_Sensor-), J?.B33 (Crank_and_Cam_Position_Sensors-), J?.D28 (Accel_Position_1_GND), J?.D29 (Accel_Position_2_GND)
- no-connect marks 97 -> 45
Other:
- note added: "FIXME: Accel and TPS 2?"
- note added: "FIXME: CAN bus or Tach on wires"
- note removed: "1. A/C High Pressure Switch"
- note removed: "1. EFI2 Fuse - (after EFI Relay)"
- note removed: "1. Injector 1"
- note removed: "1. Knock Sensor+"
- note removed: "10. Fuel Pump Relay"
- note removed: "10. Ignition Coil 3"
- note removed: "11. Ignition Coil 4"
- note removed: "11. Malfunction Lamp"
- note removed: "12. Camshaft Timing Control- (VVT)"
- note removed: "12. Stop Switch Inverted"
- note removed: "12. Tail Lights Active"
- note removed: "13. Camshaft Timing Control+ (VVT)"
- note removed: "13. Rear Window Defog Active"
- note removed: "14. Comination Meter THWO"
- note removed: "14. Radiator Fan High/Low"
- note removed: "15. Power Ground"
- note removed: "16. Neutral Safety Switch"
- note removed: "16. Radiator Fan On/Off"
- note removed: "17. ABS/Skid NEO"
- note removed: "17. Drive-by-Wire Motor Shield"
- note removed: "17. Speed Signal"
- note removed: "17. Starting Signal"
- note removed: "18. Data Link SIL"
- note removed: "18. Throttle Sensor Power"
- note removed: "19. Coolant Temp Sensor"
- note removed: "19. Data Link WFSE"
- note removed: "19. Stop Lamp Active"
- note removed: "2. AC Mag Clutch Relay"
- note removed: "2. Injector 2"
- note removed: "2. Power Ground"
- note removed: "20. Data Link TC"
- note removed: "20. MAF Thermistor"
- note removed: "21. Canister Pump Pressure Sensor"
- note removed: "21. O2 Bank 1 Sensor 2 Heater"
- note removed: "21. Throttle Body Position Sensor 1"
- note removed: "22. Accel Position 1 Signal"
- note removed: "23. Accel Position 2 Signal"
- note removed: "23. O2 Bank 1 Sensor 1 Signal+"
- note removed: "24. ABS/Skid ENG+"
- note removed: "24. Camshaft Position Sensor+"
- note removed: "24. Cruise Control Input"
- note removed: "24. Ignition Coil Feedback"
- note removed: "25. ABS/Skid VSC+"
- note removed: "25. Crankshaft Position Sensor+"
- note removed: "26. Accel Position 1 V+"
- note removed: "26. Transponder Key Module B"
- note removed: "27. Accel Position 2 V+"
- note removed: "27. Canister Pump Vent Valve"
- note removed: "27. Transponder Key Module W"
- note removed: "28. A/C Enable SW"
- note removed: "28. Accel Position 1 GND"
- note removed: "28. Knock Sensor-"
- note removed: "28. Signal Ground"
- note removed: "29. Accel Position 2 GND"
- note removed: "29. MAF Air Flow EVG"
- note removed: "29. O2 Bank 1 Sensor 2 Signal"
- note removed: "3. Drive-by-Wire Motor-"
- note removed: "3. EFI Fuse - Battery"
- note removed: "3. Injector 3"
- note removed: "30. ABS/Skid ENG-"
- note removed: "30. MAF Air Flow VG"
- note removed: "31. ABS/Skid VSC-"
- note removed: "31. O2 Bank 1 Sensor 1 Signal-"
- note removed: "31. Throttle Body Position Sensor 2"
- note removed: "32. A/C Evap Thermistor"
- note removed: "33. A/C SW Indicator"
- note removed: "33. Crank and Cam Position Sensors-"
- note removed: "34. VSV (Purge)"
- note removed: "35. Chassis Ground"
- note removed: "4. Canister Pump Motor Power"
- note removed: "4. Drive-by-Wire Motor+"
- note removed: "4. Injector 4"
- note removed: "5. O2 Bank 1 Sensor 1 Heater"
- note removed: "5. Signal Shielding Ground"
- note removed: "5. Tachometer Output"
- note removed: "6. ETCS Fuse - Battery"
- note removed: "6. Power Ground"
- note removed: "7. Power Ground"
- note removed: "8. EFI Relay"
- note removed: "8. Ignition Coil 1"
- note removed: "8. Power Steering Fluid Low"
- note removed: "9. Ignition Coil 2"
- note removed: "9. Ignition Switch"
- note removed: "NOTE: Link for A/C Indicator"
- note removed: "NOTE: Link for Shielding"
