File: Lotus Elise 2005 Stock Harness to EMU Black/Lotus Elise 2005 Stock Harness to EMU Black.kicad_sch (KiCad schematic)
At the start: 5 parts, among them J1 ECU Black - Black Connector, J2 ECU Black - Grey Connector, J3 Lotus Elise 2005 - No DBW - E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, J4 Lotus Elise 2005 - No DBW - E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, J5 Wide Band O2 - Bosch 4.9

Commit message: Added more nets
Connections:
- net VVL Solenoid: now reaches J4.12 (VVL_Oil_Valve_Out)
- net VVL Solenoid: now also J2.12 (AUX_5)
- net Knock_Sig: now reaches J4.13 (Knock_Sens_Sig_Gnd)
- net Knock_Sig: now also J1.3 (Knock_Sensor_In_1)
- net Cam Sig: now reaches J4.16 (Cam_Pos_Sens_Sig)
- net Cam Sig: now also J1.21 (Camsync_In_1)
- net Sig Gnd 29: now reaches J4.19 (Knock_Sens_Shield)
- net Sig Gnd 29: now also J1.29 (Sensor_Ground)
- net ECU Gnd: now reaches J4.2 (ECU_Gnd)
- net ECU Gnd: now also J1.28 (ECU_Ground)
- net TPS Sig: now reaches J4.20 (TPS_Sig_In)
- net TPS Sig: now also J1.18 (TPS_In)
- net VVTL Oil Sw: now reaches J4.21 (VVTL_Oil_Pres_Sw_In)
- net VVTL Oil Sw: now also J1.10 (Switch_1_In)
- net Oil Pres Sig: now reaches J4.24 (Oil_Pres_Sw_In)
- net Oil Pres Sig: now also J1.4 (Analog_In_2)
- net Power Gnd: now reaches J4.28 (ECU_Gnd)
- net Power Gnd: now also J1.27 (Power_Ground), J2.17 (Power_Ground), J2.24 (Power_Ground), J3.66 (Start_Rly_Out)
- net Coolant Temp Sig: now reaches J4.33 (Coolant_Temp_Sens_Sig_In)
- net Coolant Temp Sig: now also J1.5 (CLT_In)
- net IAC Sig: now reaches J4.35 (IAC_Sig_Out)
- net IAC Sig: now also J2.5 (AUX_3)
- net Crank Sig: now reaches J4.4 (Crank_Sens_Sig_In)
- net Crank Sig: now also J1.8 (Primary_Trigger)
- net IAT Super: now reaches J4.44 (TMAF_Sens_IAT_Sig_In)
- net IAT Super: now also J1.32 (IAT_In)
- net VVT Solenoid: now reaches J4.49 (VVT_Oil_Valve_Out)
- net VVT Solenoid: now also J2.4 (AUX_6)
- net 5V Ref 26: now reaches J4.8 (TPS_5V_Ref)
- net 5V Ref 26: now also J1.26 (5V_Supply), J3.55 (Fuel_&_VAP_5V_Ref)
- net WBO Ip: now reaches J5.1 (WBO_Ip)
- net WBO Ip: now also J1.19 (WBO_Ip)
- net WBO Vgnd: now reaches J5.2 (WBO_Sig_Gnd)
- net WBO Vgnd: now also J1.33 (WBO_VGND)
- net WBO Heater Gnd: now reaches J5.3 (WBO_Heater_Gnd)
- net WBO Heater Gnd: now also J2.19 (WBO_Heater)
- net WBO Rcal: now reaches J5.5 (WBO_Rcal)
- net WBO Rcal: now also J1.22 (WBO_Rcal)
- net WBO Vs: now reaches J5.6 (WBO_Vs)
- net WBO Vs: now also J1.6 (WBO_Vs)
- net CAN High: now reaches J1.12 (CAN_H)
- net CAN High: now also J3.65 (OBDII_CAN_High)
- net 12V Battery: now reaches J1.13 (Battery_12V)
- net 12V Battery: now also J3.80 (12V_Battery)
- net Oil Temp: now reaches J1.17 (Analog_In_3)
- net Speed Sig: now reaches J1.20 (VSS_In)
- net Speed Sig: now also J3.63 (ABS_SPD_Right_Front)
- net A/C Pres Safety: now reaches J1.23 (Switch_2_In)
- net A/C Pres Safety: now also J3.56 (A/C_Safety_Trinary_Sw_In)
- net CAN Low: now reaches J1.25 (CAN_L)
- net CAN Low: now also J3.79 (OBDII_CAN_LOW)
- net IAT Intake: now reaches J1.30 (Analog_In_4)
- net Fuel Level: now reaches J1.31 (Analog_In_1)
- net Fuel Level: now also J3.76 (Fuel_Level_Sig_In)
- net 5V Ref 34: now reaches J1.34 (5V_Supply)
- net Ext Baro: now reaches J1.35 (Analog_In_5)
- net A/C Pres Cycle: now reaches J1.36 (Switch_3_In)
- net A/C Pres Cycle: now also J3.70 (A/C_Cycle_Trinary_Sw_In)
- net Fuel Pres: now reaches J1.37 (Analog_In_6)
- net Flex Fuel Sig: now reaches J1.9 (Flex_Fuel_In)
- net A/C Clutch: now reaches J3.53 (A/C_Clutch_Out)
- net A/C Clutch: now also J2.2 (H-Bridge_1_Winding_A)
- net Engine Enable: now reaches J3.54 (Engine_Cont_Rly_Out)
- net Engine Enable: now also J2.20 (AUX_4_/_Tachometer)
- net Rad Fan 2: now reaches J3.60 (Rad_Fan_2_Rly_Out)
- net Rad Fan 2: now also J2.11 (H-Bridge_2_Winding_B)
- net 12V Ignition: now reaches J3.61 (12V_Switched_Ign)
- net 12V Ignition: now also J2.18 (Ignition_12V)
- net Rad Fan 1: now reaches J3.67 (Rad_Fan_1_Rly_Out)
- net Rad Fan 1: now also J2.3 (H-Bridge_2_Winding_A)
- net Fuel Pump: now reaches J3.68 (Fuel_Pump_Rly_Out)
- net Fuel Pump: now also J2.21 (AUX_1_/_Injector_7)
- net Hot Soak Pump: now reaches J3.69 (Hot_Soak_Pump_Rly_Out)
- net Hot Soak Pump: now also J2.10 (H-Bridge_1_Winding_B)
- net Oil Cooler Fan: now reaches J2.13 (AUX_2_/_Injector_8)
- net Fifth Injector: now reaches J2.14 (Injector_5)
- no-connect marks 0 -> 30
